File: pcb/junyapad.kicad_pcb (KiCad board)
At the start: 2 copper layers, 92.9 x 52.4 mm, 37 parts, among them J1 OLED_128x32, SW1 SW_Push_45deg, SW2 SW_Push_45deg, SW3 SW_Push_45deg, SW4 SW_Push_45deg, SW5 SW_Push_45deg, SW6 SW_Push_45deg, SW9 RotaryEncoder_Switch, U1 XIAO-RP2040-DIP

Commit message: Rearrange Capacitors
Parts:
- moved C5 57.1 mm to (219.1, 114.3), turned to 180 degrees
- moved C9 53.6 mm to (204.8, 131.1), turned to 90 degrees
- moved C7 50.1 mm to (204.8, 104.7), turned to -90 degrees
- moved C4 42.9 mm to (204.8, 109.5), turned to -90 degrees
- moved C3 38.4 mm to (200.0, 114.3), turned to 180 degrees
- moved C8 37.7 mm to (185.7, 131.1), turned to 90 degrees
- moved C6 31.0 mm to (185.7, 104.7), turned to -90 degrees
- moved C2 23.9 mm to (185.7, 109.4), turned to -90 degrees
- moved C1 21.3 mm to (181.0, 114.3), turned to 180 degrees
- moved C10 8.59 mm to (159.5, 107.2), turned to 90 degrees
