File: pcb/junyapad.kicad_pcb (KiCad board)
At the start: 2 copper layers, 92.9 x 52.4 mm, 37 parts, among them J1 OLED_128x32, SW1 SW_Push_45deg, SW2 SW_Push_45deg, SW3 SW_Push_45deg, SW4 SW_Push_45deg, SW5 SW_Push_45deg, SW6 SW_Push_45deg, SW9 RotaryEncoder_Switch, U1 XIAO-RP2040-DIP

Commit message: Export CAD files
Parts:
- added G***: LOGO, LOGO, F.Cu at (157.0, 127.5)
- added G***: LOGO, LOGO, B.Cu at (205.7, 123.0)
- added G***: LOGO, LOGO, F.Cu at (154.0, 107.0)
- added G***: LOGO, LOGO, F.Cu at (143.5, 88.5)
- added G***: LOGO, LOGO, F.Cu at (185.5, 112.5)
- added G***: LOGO, LOGO, F.Cu at (159.5, 116.5)
- added G***: LOGO, LOGO, F.Cu at (140.0, 106.0)
- added G***: LOGO, LOGO, B.Cu at (208.0, 100.5)
- added G***: LOGO, LOGO, B.Cu at (180.5, 86.0)
- added G***: LOGO, LOGO, B.Cu at (157.3, 107.3)
- moved D2 9.18 mm to (135.5, 112.5)
- moved D4 9.18 mm to (138.5, 112.5)
- moved D6 9.18 mm to (141.5, 112.5)
- moved D1 9.18 mm to (144.5, 112.5)
- moved D3 9.18 mm to (147.5, 112.5)
- moved D5 9.18 mm to (150.5, 112.5)
Routing:
- net +5V: track 0.00 -> 240.5 mm, vias 0 -> 4
- net COL2: track 0.00 -> 123.6 mm, vias 0 -> 3
- net Net-(D12-DOUT): track 0.00 -> 95.0 mm, vias 0 -> 2
- net COL1: track 0.00 -> 93.3 mm, vias 0 -> 3
- net Net-(D5-A): track 0.00 -> 88.4 mm
- net Net-(D6-A): track 0.00 -> 81.2 mm
- net EC11/SW: track 0.00 -> 75.9 mm, vias 0 -> 2
- net COL0: track 0.00 -> 73.6 mm, vias 0 -> 1
- net Net-(D3-A): track 0.00 -> 72.4 mm
- net EC11/DT: track 0.00 -> 69.4 mm, vias 0 -> 2
- net EC11/CLK: track 0.00 -> 67.0 mm, vias 0 -> 2
- net Net-(D4-A): track 0.00 -> 65.2 mm
- net Net-(D1-A): track 0.00 -> 56.3 mm
- net OLED/SCL: track 0.00 -> 49.3 mm, vias 0 -> 2
- net Net-(D2-A): track 0.00 -> 48.3 mm
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- added copper zone on B.Cu, net GND
- added copper zone on F.Cu, net GND
Other:
- outline, holes or cut-outs redrawn
- board text added: "XIAO HERE!"
- board text added: "junyali 2025-07-01"
